Commit message: Restore Changes : Robot movement to pose

File: vsss_simulation/urdf/robot.urdf.xacro (robot description, xacro)
@@ -1,4 +1,5 @@
 <robot xmlns:xacro="http://ros.org/wiki/xacro" name="vsss_robot">
     <!-- Parameters -->
+    <xacro:arg name='robot_name' default="robot"/>
     <xacro:property name="wheel_radius" value="0.05"/>
     <xacro:property name="wheel_width" value="0.02"/>
@@ -6,5 +7,5 @@
     <xacro:property name="body_size" value="0.3"/>
     <!-- Base Link -->
-    <link name="base_link">
+    <link name="$(arg robot_name)_base_link">
         <visual>
             <origin xyz="0 0 ${body_size / 2}" rpy="0 0 0"/>
@@ -108,5 +109,5 @@
     <!-- Wheel Joints -->
     <joint name="left_wheel_joint" type="continuous">
-        <parent link="base_link"/>
+        <parent link="$(arg robot_name)_base_link"/>
         <child link="left_wheel_link"/>
         <origin xyz="0 -${wheel_separation/2} 0" rpy="1.57 0 0"/>
@@ -114,5 +115,5 @@
     </joint>
     <joint name="right_wheel_joint" type="continuous">
-        <parent link="base_link"/>
+        <parent link="$(arg robot_name)_base_link"/>
         <child link="right_wheel_link"/>
         <origin xyz="0 ${wheel_separation/2} 0" rpy="1.57 0 0"/>
@@ -120,5 +121,5 @@
     </joint>
     <joint name="dominant_plate_joint" type="fixed">
-        <parent link="base_link"/>
+        <parent link="$(arg robot_name)_base_link"/>
         <child link="dominant_plate_link"/>
         <origin xyz="${-body_size / 4} 0.0 ${body_size + 0.01}" rpy="0.0 0.0 0.0"/>
@@ -126,5 +127,5 @@
     </joint>
     <joint name="small_plate_1_joint" type="fixed">
-        <parent link="base_link"/>
+        <parent link="$(arg robot_name)_base_link"/>
         <child link="small_plate_1_link"/>
         <origin xyz="${body_size / 4} ${body_size / 4} ${body_size + 0.01}" rpy="0.0 0.0 0.0"/>
@@ -132,5 +133,5 @@
     </joint>
     <joint name="small_plate_2_joint" type="fixed">
-        <parent link="base_link"/>
+        <parent link="$(arg robot_name)_base_link"/>
         <child link="small_plate_2_link"/>
         <origin xyz="${body_size / 4} ${-body_size / 4} ${body_size + 0.01}" rpy="0.0 0.0 0.0"/>
@@ -152,5 +153,8 @@
     <!-- Gazebo Diff Drive Plugin -->
     <gazebo>
-        <plugin name="diff_drive_controller" filename="libgazebo_ros_diff_drive.so">
+        <plugin name="$(arg robot_name)_diff_drive_controller" filename="libgazebo_ros_diff_drive.so">
+        <ros>
+            <namespace>/$(arg robot_name)</namespace>
+        </ros>
             <left_joint>left_wheel_joint</left_joint>
             <right_joint>right_wheel_joint</right_joint>
@@ -161,9 +165,9 @@
             <odom_topic>odom</odom_topic>
             <cmd_vel_topic>cmd_vel</cmd_vel_topic>
-            <robot_base_frame>base_link</robot_base_frame>
+            <robot_base_frame>$(arg robot_name)_base_link</robot_base_frame>
         </plugin>
     </gazebo>
     <!-- Gazebo Material -->
-    <gazebo reference="base_link">
+    <gazebo reference="$(arg robot_name)_base_link">
         <material>Gazebo/Black</material>
     </gazebo>
