Commit message: feat: change object models

File: vsss/vsss_simulation/urdf/robot.urdf.xacro (robot description, xacro)
@@ -2,4 +2,7 @@
     <!-- Parameters -->
     <xacro:arg name='robot_name' default="robot"/>
+    <xacro:arg name='dominant_plate_color' default="BlueLaser"/>
+    <xacro:arg name='small_plate_1' default="Green"/>
+    <xacro:arg name='small_plate_2' default="Turquoise"/>
     <xacro:property name="wheel_radius" value="0.05"/>
     <xacro:property name="wheel_width" value="0.02"/>
@@ -179,11 +182,11 @@
     </gazebo>
     <gazebo reference="dominant_plate_link">
-        <material>Gazebo/Yellow</material>
+        <material>Gazebo/$(arg dominant_plate_color)</material>
     </gazebo>
     <gazebo reference="small_plate_1_link">
-        <material>Gazebo/Green</material>
+        <material>Gazebo/$(arg small_plate_1)</material>
     </gazebo>
     <gazebo reference="small_plate_2_link">
-        <material>Gazebo/Pink</material>
+        <material>Gazebo/$(arg small_plate_2)</material>
     </gazebo>
 </robot>

Commit message: Docker Functionality <> Polygon Class

File: vsss/vsss_simulation/urdf/robot.urdf.xacro (robot description, xacro)
@@ -27,5 +27,6 @@
         </collision>
         <inertial>
-            <mass value="1.0"/>
+            <origin xyz="0 0 -0.01"/>
+            <mass value="3.5"/>
             <inertia ixx="0.01" ixy="0.0" ixz="0.0" iyy="0.01" iyz="0.0" izz="0.01"/>
         </inertial>
